File: pcb/esp8266-programmer.brd (EAGLE design)
At the start: 45.7 x 25.4 mm, 14 parts

Commit message: Final board design.
Parts:
- C3: device rcl:C/6032-28R -> rcl:A/3216-18W
Routing:
- net +5V: track 42.0 -> 42.9 mm
Changed lines of the file:
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@@
 <wire x1="0" y1="22.86" x2="0" y2="2.54" width="0" layer="20"/>
 <wire x1="0" y1="2.54" x2="2.54" y2="0" width="0" layer="20" curve="90"/>
-<text x="19.304" y="19.558" size="1.778" layer="25" font="vector" ratio="15" rot="R90">3V3</text>
-<text x="29.21" y="20.32" size="1.778" layer="25" font="vector" ratio="15" rot="R90">5V</text>
-<text x="29.464" y="11.684" size="1.016" layer="26" font="vector" ratio="15" rot="MR0">ivo.slanina@gmail.com</text>
-<text x="29.464" y="13.208" size="1.143" layer="26" font="vector" ratio="15" rot="MR0">ESP8266 PROGRAMMER v0.1.0</text>
+<text x="19.304" y="21.844" size="1.778" layer="25" font="vector" ratio="15" rot="R90" align="bottom-center">3V3</text>
+<text x="27.432" y="21.844" size="1.778" layer="25" font="vector" ratio="15" rot="R90" align="top-center">5V</text>
+<text x="29.464" y="11.684" size="1.016" layer="22" font="vector" ratio="15" rot="MR0">ivo.slanina@gmail.com</text>
+<text x="29.464" y="13.208" size="1.143" layer="22" font="vector" ratio="15" rot="MR0">ESP8266 PROGRAMMER v0.1.0</text>
 </plain>
 <attributes>
@@
 <attribute name="VALUE" x="13.716" y="21.082" size="1.27" layer="27" rot="R270"/>
 </element>
-<element name="C3" library="rcl" package="C/6032-28R" value="10uF" x="11.176" y="20.574" smashed="yes" rot="R270">
-<attribute name="NAME" x="9.351" y="19.86" size="1.27" layer="25" font="vector" ratio="15" rot="R90"/>
+<element name="C3" library="rcl" package="A/3216-18W" value="10uF" x="11.176" y="20.574" smashed="yes" rot="R270">
+<attribute name="NAME" x="9.605" y="19.86" size="1.27" layer="25" font="vector" ratio="15" rot="R90"/>
 <attribute name="VALUE" x="8.126" y="23.574" size="1.27" layer="27" rot="R270"/>
 </element>
@@
 <via x="43.688" y="1.524" extent="1-16" drill="0.5"/>
 <via x="44.45" y="12.7" extent="1-16" drill="0.5"/>
+<via x="15.494" y="5.588" extent="1-16" drill="0.5"/>
+<via x="31.75" y="8.89" extent="1-16" drill="0.5"/>
 </signal>
 <signal name="TXD">
@@
 <wire x1="22.311" y1="13.167" x2="25.908" y2="16.764" width="0.4064" layer="1"/>
 <wire x1="25.908" y1="16.764" x2="25.908" y2="21.844" width="0.4064" layer="1"/>
-<wire x1="11.176" y1="18.049" x2="11.176" y2="16.256" width="0.4064" layer="1"/>
+<wire x1="11.176" y1="19.099" x2="11.176" y2="16.256" width="0.4064" layer="1"/>
 <wire x1="11.176" y1="16.256" x2="11.684" y2="15.748" width="0.4064" layer="1"/>
-<wire x1="11.176" y1="18.049" x2="13.157" y2="18.049" width="0.4064" layer="1"/>
-<wire x1="13.157" y1="18.049" x2="13.97" y2="18.862" width="0.4064" layer="1"/>
+<wire x1="11.176" y1="19.099" x2="13.97" y2="19.099" width="0.4064" layer="1"/>
+<wire x1="13.97" y1="19.099" x2="13.97" y2="18.862" width="0.4064" layer="1"/>
 </signal>
 <signal name="USBDM">
